Commit message: Add P3020 Descriptions (#166)
* Add P3020 Model description (with moveit, gazebo, rviz launch).

* Update Docker Emulator with robot model argument.

* Update nodes, controller and sim_time for Gazebo Handling.

File: dsr_description2/config/macro.gazebo.p3020.xacro (robot description, xacro)
@@ -9,5 +9,5 @@
           <namespace>$(arg namespace)</namespace>
         </ros>
-        <parameters>$(find dsr_controller2)/config/dsr_controller2_gz.yaml</parameters>
+        <parameters>$(find dsr_controller2)/config/dsr_controller2_gz_p3020.yaml</parameters>
       </plugin>
     </gazebo>

File: dsr_description2/config/macro.materials.xacro (robot description, xacro)
@@ -17,4 +17,7 @@
 			<color rgba="0.941 0.941 0.941 1.0" />
 		</material>
+		<material name="dr_blue">
+			<color rgba="0 0 0.15 1" />
+		</material>
 	</xacro:macro>
 </robot>
