Commit message: Use xacro.load_yaml syntax to remove warnings (#179) (#182)
* Use xacro.load_yaml to remove warnings
* Fix missing base link in h2017.urdf

Co-authored-by: Bent Martin Dyrdal <70641282+bmdyrdal@users.noreply.github.com>

File: dsr_description2/urdf/h2017.urdf (robot description, URDF)
Before this commit: robot h2017, 8 links, 8 joints
Links:
- added link base

File: dsr_moveit2/dsr_moveit_config_a0509/config/dsr.ros2_control.xacro (robot description, xacro)
@@ -2,5 +2,5 @@
 <robot xmlns:xacro="http://www.ros.org/wiki/xacro">
     <xacro:macro name="dsr_moveit_ros2_control" params="name initial_positions_file">
-        <xacro:property name="initial_positions" value="${load_yaml(initial_positions_file)['initial_positions']}"/>
+        <xacro:property name="initial_positions" value="${xacro.load_yaml(initial_positions_file)['initial_positions']}"/>
         <ros2_control name="${name}" type="system">
             <hardware>

File: dsr_moveit2/dsr_moveit_config_m1013/config/dsr.ros2_control.xacro (robot description, xacro)
@@ -2,5 +2,5 @@
 <robot xmlns:xacro="http://www.ros.org/wiki/xacro">
     <xacro:macro name="dsr_moveit_ros2_control" params="name initial_positions_file">
-        <xacro:property name="initial_positions" value="${load_yaml(initial_positions_file)['initial_positions']}"/>
+        <xacro:property name="initial_positions" value="${xacro.load_yaml(initial_positions_file)['initial_positions']}"/>
         <ros2_control name="${name}" type="system">
             <hardware>

File: dsr_moveit2/dsr_moveit_config_p3020/config/dsr.ros2_control.xacro (robot description, xacro)
@@ -2,5 +2,5 @@
 <robot xmlns:xacro="http://www.ros.org/wiki/xacro">
     <xacro:macro name="dsr_moveit_ros2_control" params="name initial_positions_file">
-        <xacro:property name="initial_positions" value="${load_yaml(initial_positions_file)['initial_positions']}"/>
+        <xacro:property name="initial_positions" value="${xacro.load_yaml(initial_positions_file)['initial_positions']}"/>
         <ros2_control name="${name}" type="system">
             <hardware>
