Commit message: Remove all tool0 links in urdf (#195)
Removed tool0 from the URDF as it's not used in the provided launches.

File: dsr_description2/urdf/a0509.urdf (robot description, URDF)
Before this commit: robot a0509, 9 links, 8 joints
Links:
- removed link tool0
Joints:
- removed joint joint_6-tool0

File: dsr_description2/urdf/a0912.urdf (robot description, URDF)
Before this commit: robot a0912, 9 links, 8 joints
Links:
- removed link tool0
Joints:
- removed joint joint_6-tool0

File: dsr_description2/urdf/e0509.urdf (robot description, URDF)
Before this commit: robot e0509, 9 links, 8 joints
Links:
- removed link tool0
Joints:
- removed joint joint_6-tool0

File: dsr_description2/urdf/h2017.urdf (robot description, URDF)
Before this commit: robot h2017, 9 links, 8 joints
Links:
- removed link tool0
Joints:
- removed joint joint_6-tool0

File: dsr_description2/urdf/h2515.urdf (robot description, URDF)
Before this commit: robot h2515, 9 links, 8 joints
Links:
- removed link tool0
Joints:
- removed joint joint_6-tool0

File: dsr_description2/urdf/m0609.urdf (robot description, URDF)
Before this commit: robot m0609, 9 links, 8 joints
Links:
- removed link tool0
Joints:
- removed joint joint_6-tool0

File: dsr_description2/urdf/m0617.urdf (robot description, URDF)
Before this commit: robot m0617, 9 links, 8 joints
Links:
- removed link tool0
Joints:
- removed joint joint_6-tool0

File: dsr_description2/urdf/m1013.urdf (robot description, URDF)
Before this commit: robot m1013, 9 links, 8 joints
Links:
- removed link tool0
Joints:
- removed joint joint_6-tool0

File: dsr_description2/urdf/m1509.urdf (robot description, URDF)
Before this commit: robot m1509, 9 links, 8 joints
Links:
- removed link tool0
Joints:
- removed joint joint_6-tool0
