Commit message: fixed urdf with tool for M1013, M0609 (#230)

File: dsr_description2/urdf/m0609.urdf (robot description, URDF)
Before this commit: robot m0609, 8 links, 7 joints
Links:
- added link tool0
Joints:
- added joint joint_6-tool0: type fixed, parent link_6, child tool0, origin xyz=0 0 0 rpy=3.1415926535 -1.570796327 0

File: dsr_description2/urdf/m1013.urdf (robot description, URDF)
Before this commit: robot m1013, 8 links, 7 joints
Links:
- added link tool0
Joints:
- added joint joint_6-tool0: type fixed, parent link_6, child tool0, origin xyz=0 0 0 rpy=3.1415926535 -1.570796327 0
