Commit message: Refactor controller  (#215)
* Refactor hw_interface & dsr_controller

* Fix launches as being changed workaround param to the standard way

File: dsr_description2/ros2_control/a0509.ros2_control.xacro (robot description, xacro)
@@ -3,27 +3,18 @@
   <xacro:macro name="a0509_ros2_control" params="
   name
-  rate:=100
-  standby:=ture
-  command:=none
   host:=0.0.0.0
+  rt_host:=0.0.0.0
   port:=12345
   mode:=real
   model:=a0509
-  gripper:=none
-  mobile:=none
   ">
     <ros2_control name="${name}" type="system">
       <hardware>
         <plugin>dsr_hardware2/DRHWInterface</plugin>
-        <param name="name">${name}</param>
-        <param name="rate">${rate}</param>
-        <param name="standby">${standby}</param>
-        <param name="command">${command}</param>
         <param name="host">${host}</param>
+        <param name="rt_host">${rt_host}</param>
         <param name="port">${port}</param>
         <param name="mode">${mode}</param>
         <param name="model">${model}</param>
-        <param name="gripper">${gripper}</param>
-        <param name="mobile">${mobile}</param>
       </hardware>
       <joint name="joint_1">

File: dsr_description2/ros2_control/a0912.ros2_control.xacro (robot description, xacro)
@@ -3,27 +3,18 @@
   <xacro:macro name="a0912_ros2_control" params="
   name
-  rate:=100
-  standby:=ture
-  command:=none
   host:=0.0.0.0
+  rt_host:=0.0.0.0
   port:=12345
   mode:=real
   model:=a0912
-  gripper:=none
-  mobile:=none
   ">
     <ros2_control name="${name}" type="system">
       <hardware>
         <plugin>dsr_hardware2/DRHWInterface</plugin>
-        <param name="name">${name}</param>
-        <param name="rate">${rate}</param>
-        <param name="standby">${standby}</param>
-        <param name="command">${command}</param>
         <param name="host">${host}</param>
+        <param name="rt_host">${rt_host}</param>
         <param name="port">${port}</param>
         <param name="mode">${mode}</param>
         <param name="model">${model}</param>
-        <param name="gripper">${gripper}</param>
-        <param name="mobile">${mobile}</param>
       </hardware>
       <joint name="joint_1">

File: dsr_description2/ros2_control/e0509.ros2_control.xacro (robot description, xacro)
@@ -3,27 +3,18 @@
   <xacro:macro name="e0509_ros2_control" params="
   name
-  rate:=100
-  standby:=ture
-  command:=none
   host:=0.0.0.0
+  rt_host:=0.0.0.0
   port:=12345
   mode:=real
   model:=e0509
-  gripper:=none
-  mobile:=none
   ">
     <ros2_control name="${name}" type="system">
       <hardware>
         <plugin>dsr_hardware2/DRHWInterface</plugin>
-        <param name="name">${name}</param>
-        <param name="rate">${rate}</param>
-        <param name="standby">${standby}</param>
-        <param name="command">${command}</param>
         <param name="host">${host}</param>
+        <param name="rt_host">${rt_host}</param>
         <param name="port">${port}</param>
         <param name="mode">${mode}</param>
         <param name="model">${model}</param>
-        <param name="gripper">${gripper}</param>
-        <param name="mobile">${mobile}</param>
       </hardware>
       <joint name="joint_1">

File: dsr_description2/ros2_control/h2017.ros2_control.xacro (robot description, xacro)
@@ -3,27 +3,18 @@
   <xacro:macro name="h2017_ros2_control" params="
   name
-  rate:=100
-  standby:=ture
-  command:=none
   host:=0.0.0.0
+  rt_host:=0.0.0.0
   port:=12345
   mode:=real
   model:=h2017
-  gripper:=none
-  mobile:=none
   ">
     <ros2_control name="${name}" type="system">
       <hardware>
         <plugin>dsr_hardware2/DRHWInterface</plugin>
-        <param name="name">${name}</param>
-        <param name="rate">${rate}</param>
-        <param name="standby">${standby}</param>
-        <param name="command">${command}</param>
         <param name="host">${host}</param>
+        <param name="rt_host">${rt_host}</param>
         <param name="port">${port}</param>
         <param name="mode">${mode}</param>
         <param name="model">${model}</param>
-        <param name="gripper">${gripper}</param>
-        <param name="mobile">${mobile}</param>
       </hardware>
       <joint name="joint_1">

File: dsr_description2/ros2_control/h2515.ros2_control.xacro (robot description, xacro)
@@ -3,27 +3,18 @@
   <xacro:macro name="h2515_ros2_control" params="
   name
-  rate:=100
-  standby:=ture
-  command:=none
   host:=0.0.0.0
+  rt_host:=0.0.0.0
   port:=12345
   mode:=real
   model:=h2515
-  gripper:=none
-  mobile:=none
   ">
     <ros2_control name="${name}" type="system">
       <hardware>
         <plugin>dsr_hardware2/DRHWInterface</plugin>
-        <param name="name">${name}</param>
-        <param name="rate">${rate}</param>
-        <param name="standby">${standby}</param>
-        <param name="command">${command}</param>
         <param name="host">${host}</param>
+        <param name="rt_host">${rt_host}</param>
         <param name="port">${port}</param>
         <param name="mode">${mode}</param>
         <param name="model">${model}</param>
-        <param name="gripper">${gripper}</param>
-        <param name="mobile">${mobile}</param>
       </hardware>
       <joint name="joint_1">

File: dsr_description2/ros2_control/m0609.ros2_control.xacro (robot description, xacro)
@@ -3,27 +3,18 @@
   <xacro:macro name="m0609_ros2_control" params="
   name
-  rate:=100
-  standby:=ture
-  command:=none
   host:=0.0.0.0
+  rt_host:=0.0.0.0
   port:=12345
   mode:=real
   model:=m0609
-  gripper:=none
-  mobile:=none
   ">
     <ros2_control name="${name}" type="system">
       <hardware>
         <plugin>dsr_hardware2/DRHWInterface</plugin>
-        <param name="name">${name}</param>
-        <param name="rate">${rate}</param>
-        <param name="standby">${standby}</param>
-        <param name="command">${command}</param>
         <param name="host">${host}</param>
+        <param name="rt_host">${rt_host}</param>
         <param name="port">${port}</param>
         <param name="mode">${mode}</param>
         <param name="model">${model}</param>
-        <param name="gripper">${gripper}</param>
-        <param name="mobile">${mobile}</param>
       </hardware>
       <joint name="joint_1">

File: dsr_description2/ros2_control/m0617.ros2_control.xacro (robot description, xacro)
@@ -3,27 +3,18 @@
   <xacro:macro name="m0617_ros2_control" params="
   name
-  rate:=100
-  standby:=ture
-  command:=none
   host:=0.0.0.0
+  rt_host:=0.0.0.0
   port:=12345
   mode:=real
   model:=m0617
-  gripper:=none
-  mobile:=none
   ">
     <ros2_control name="${name}" type="system">
       <hardware>
         <plugin>dsr_hardware2/DRHWInterface</plugin>
-        <param name="name">${name}</param>
-        <param name="rate">${rate}</param>
-        <param name="standby">${standby}</param>
-        <param name="command">${command}</param>
         <param name="host">${host}</param>
+        <param name="rt_host">${rt_host}</param>
         <param name="port">${port}</param>
         <param name="mode">${mode}</param>
         <param name="model">${model}</param>
-        <param name="gripper">${gripper}</param>
-        <param name="mobile">${mobile}</param>
       </hardware>
       <joint name="joint_1">

File: dsr_description2/ros2_control/m1013.ros2_control.xacro (robot description, xacro)
@@ -3,27 +3,18 @@
   <xacro:macro name="m1013_ros2_control" params="
   name
-  rate:=100
-  standby:=ture
-  command:=none
   host:=0.0.0.0
+  rt_host:=0.0.0.0
   port:=12345
   mode:=real
   model:=m1013
-  gripper:=none
-  mobile:=none
   ">
     <ros2_control name="${name}" type="system">
       <hardware>
         <plugin>dsr_hardware2/DRHWInterface</plugin>
-        <param name="name">${name}</param>
-        <param name="rate">${rate}</param>
-        <param name="standby">${standby}</param>
-        <param name="command">${command}</param>
         <param name="host">${host}</param>
+        <param name="rt_host">${rt_host}</param>
         <param name="port">${port}</param>
         <param name="mode">${mode}</param>
         <param name="model">${model}</param>
-        <param name="gripper">${gripper}</param>
-        <param name="mobile">${mobile}</param>
       </hardware>
       <joint name="joint_1">

File: dsr_description2/ros2_control/m1509.ros2_control.xacro (robot description, xacro)
@@ -3,27 +3,18 @@
   <xacro:macro name="m1509_ros2_control" params="
   name
-  rate:=100
-  standby:=ture
-  command:=none
   host:=0.0.0.0
+  rt_host:=0.0.0.0
   port:=12345
   mode:=real
   model:=m1509
-  gripper:=none
-  mobile:=none
   ">
     <ros2_control name="${name}" type="system">
       <hardware>
         <plugin>dsr_hardware2/DRHWInterface</plugin>
-        <param name="name">${name}</param>
-        <param name="rate">${rate}</param>
-        <param name="standby">${standby}</param>
-        <param name="command">${command}</param>
         <param name="host">${host}</param>
+        <param name="rt_host">${rt_host}</param>
         <param name="port">${port}</param>
         <param name="mode">${mode}</param>
         <param name="model">${model}</param>
-        <param name="gripper">${gripper}</param>
-        <param name="mobile">${mobile}</param>
       </hardware>
       <joint name="joint_1">

File: dsr_description2/ros2_control/p3020.ros2_control.xacro (robot description, xacro)
@@ -3,27 +3,18 @@
   <xacro:macro name="p3020_ros2_control" params="
   name
-  rate:=100
-  standby:=ture
-  command:=none
   host:=0.0.0.0
+  rt_host:=0.0.0.0
   port:=12345
   mode:=real
   model:=p3020
-  gripper:=none
-  mobile:=none
   ">
     <ros2_control name="${name}" type="system">
       <hardware>
         <plugin>dsr_hardware2/DRHWInterface</plugin>
-        <param name="name">${name}</param>
-        <param name="rate">${rate}</param>
-        <param name="standby">${standby}</param>
-        <param name="command">${command}</param>
         <param name="host">${host}</param>
+        <param name="rt_host">${rt_host}</param>
         <param name="port">${port}</param>
         <param name="mode">${mode}</param>
         <param name="model">${model}</param>
-        <param name="gripper">${gripper}</param>
-        <param name="mobile">${mobile}</param>
       </hardware>
       <joint name="joint_1">

File: dsr_description2/xacro/a0509.urdf.xacro (robot description, xacro)
@@ -5,7 +5,17 @@
   <xacro:arg name="namespace" default=""/>
   <xacro:arg name="use_gazebo" default="false"/>
+  <xacro:arg name="host" default=""/>
+  <xacro:arg name="port" default=""/>
+  <xacro:arg name="rt_host" default=""/>
+  <xacro:arg name="mode" default=""/>
+  <xacro:arg name="model" default=""/>
   <xacro:property name="cr" value="$(arg color)"/>
   <xacro:property name="gr" value="$(arg gripper)"/>
   <xacro:property name="gz" value="$(arg use_gazebo)"/>
+  <xacro:property name="host" value="$(arg host)"/>
+  <xacro:property name="rt_host" value="$(arg rt_host)"/>
+  <xacro:property name="port" value="$(arg port)"/>
+  <xacro:property name="mode" value="$(arg mode)"/>
+  <xacro:property name="model" value="$(arg model)"/>
   <xacro:if value="${cr == 'white'}">
      <xacro:include filename="$(find dsr_description2)/xacro/macro.a0509.white.xacro" />
@@ -28,5 +38,11 @@
   <xacro:unless value="${gz}">
     <xacro:include filename="$(find dsr_description2)/ros2_control/a0509.ros2_control.xacro" />
-    <xacro:a0509_ros2_control name="a0509"/>
+    <xacro:a0509_ros2_control name="a0509"
+      host="${host}"
+      rt_host="${rt_host}"
+      port="${port}"
+      mode="${mode}"
+      model="${model}"
+    />
   </xacro:unless>
 </robot>

File: dsr_description2/xacro/a0912.urdf.xacro (robot description, xacro)
@@ -5,7 +5,17 @@
   <xacro:arg name="namespace" default=""/>
   <xacro:arg name="use_gazebo" default="false"/>
+  <xacro:arg name="host" default=""/>
+  <xacro:arg name="port" default=""/>
+  <xacro:arg name="rt_host" default=""/>
+  <xacro:arg name="mode" default=""/>
+  <xacro:arg name="model" default=""/>
   <xacro:property name="cr" value="$(arg color)"/>
   <xacro:property name="gr" value="$(arg gripper)"/>
   <xacro:property name="gz" value="$(arg use_gazebo)"/>
+  <xacro:property name="host" value="$(arg host)"/>
+  <xacro:property name="rt_host" value="$(arg rt_host)"/>
+  <xacro:property name="port" value="$(arg port)"/>
+  <xacro:property name="mode" value="$(arg mode)"/>
+  <xacro:property name="model" value="$(arg model)"/>
   <xacro:if value="${cr == 'white'}">
      <xacro:include filename="$(find dsr_description2)/xacro/macro.a0912.white.xacro" />
@@ -28,5 +38,11 @@
   <xacro:unless value="${gz}">
     <xacro:include filename="$(find dsr_description2)/ros2_control/a0912.ros2_control.xacro" />
-    <xacro:a0912_ros2_control name="a0912"/>
+    <xacro:a0912_ros2_control name="a0912"
+      host="${host}"
+      rt_host="${rt_host}"
+      port="${port}"
+      mode="${mode}"
+      model="${model}"
+    />
   </xacro:unless>
 </robot>

File: dsr_description2/xacro/e0509.urdf.xacro (robot description, xacro)
@@ -5,7 +5,17 @@
   <xacro:arg name="namespace" default=""/>
   <xacro:arg name="use_gazebo" default="false"/>
+  <xacro:arg name="host" default=""/>
+  <xacro:arg name="port" default=""/>
+  <xacro:arg name="rt_host" default=""/>
+  <xacro:arg name="mode" default=""/>
+  <xacro:arg name="model" default=""/>
   <xacro:property name="cr" value="$(arg color)"/>
   <xacro:property name="gr" value="$(arg gripper)"/>
   <xacro:property name="gz" value="$(arg use_gazebo)"/>
+  <xacro:property name="host" value="$(arg host)"/>
+  <xacro:property name="rt_host" value="$(arg rt_host)"/>
+  <xacro:property name="port" value="$(arg port)"/>
+  <xacro:property name="mode" value="$(arg mode)"/>
+  <xacro:property name="model" value="$(arg model)"/>
   <xacro:if value="${cr == 'white'}">
      <xacro:include filename="$(find dsr_description2)/xacro/macro.e0509.white.xacro" />
@@ -25,5 +35,12 @@
   <xacro:unless value="${gz}">
     <xacro:include filename="$(find dsr_description2)/ros2_control/e0509.ros2_control.xacro" />
-    <xacro:e0509_ros2_control name="e0509"/>
+    <xacro:e0509_ros2_control
+      name="e0509"
+      host="${host}"
+      rt_host="${rt_host}"
+      port="${port}"
+      mode="${mode}"
+      model="${model}"
+    />
   </xacro:unless>
 </robot>

File: dsr_description2/xacro/h2017.urdf.xacro (robot description, xacro)
@@ -5,7 +5,17 @@
   <xacro:arg name="namespace" default=""/>
   <xacro:arg name="use_gazebo" default="false"/>
+  <xacro:arg name="host" default=""/>
+  <xacro:arg name="port" default=""/>
+  <xacro:arg name="rt_host" default=""/>
+  <xacro:arg name="mode" default=""/>
+  <xacro:arg name="model" default=""/>
   <xacro:property name="cr" value="$(arg color)"/>
   <xacro:property name="gr" value="$(arg gripper)"/>
   <xacro:property name="gz" value="$(arg use_gazebo)"/>
+  <xacro:property name="host" value="$(arg host)"/>
+  <xacro:property name="rt_host" value="$(arg rt_host)"/>
+  <xacro:property name="port" value="$(arg port)"/>
+  <xacro:property name="mode" value="$(arg mode)"/>
+  <xacro:property name="model" value="$(arg model)"/>
   <xacro:if value="${cr == 'white'}">
      <xacro:include filename="$(find dsr_description2)/xacro/macro.h2017.white.xacro" />
@@ -28,5 +38,12 @@
   <xacro:unless value="${gz}">
     <xacro:include filename="$(find dsr_description2)/ros2_control/h2017.ros2_control.xacro" />
-    <xacro:h2017_ros2_control name="h2017"/>
+    <xacro:h2017_ros2_control
+      name="h2017"
+      host="${host}"
+      rt_host="${rt_host}"
+      port="${port}"
+      mode="${mode}"
+      model="${model}"
+    />
   </xacro:unless>
 </robot>

File: dsr_description2/xacro/h2515.urdf.xacro (robot description, xacro)
@@ -5,7 +5,17 @@
   <xacro:arg name="namespace" default=""/>
   <xacro:arg name="use_gazebo" default="false"/>
+  <xacro:arg name="host" default=""/>
+  <xacro:arg name="port" default=""/>
+  <xacro:arg name="rt_host" default=""/>
+  <xacro:arg name="mode" default=""/>
+  <xacro:arg name="model" default=""/>
   <xacro:property name="cr" value="$(arg color)"/>
   <xacro:property name="gr" value="$(arg gripper)"/>
   <xacro:property name="gz" value="$(arg use_gazebo)"/>
+  <xacro:property name="host" value="$(arg host)"/>
+  <xacro:property name="rt_host" value="$(arg rt_host)"/>
+  <xacro:property name="port" value="$(arg port)"/>
+  <xacro:property name="mode" value="$(arg mode)"/>
+  <xacro:property name="model" value="$(arg model)"/>
   <xacro:if value="${cr == 'white'}">
      <xacro:include filename="$(find dsr_description2)/xacro/macro.h2515.white.xacro" />
@@ -28,5 +38,12 @@
   <xacro:unless value="${gz}">
     <xacro:include filename="$(find dsr_description2)/ros2_control/h2515.ros2_control.xacro" />
-    <xacro:h2515_ros2_control name="h2515"/>
+    <xacro:h2515_ros2_control
+      name="h2515"
+      host="${host}"
+      rt_host="${rt_host}"
+      port="${port}"
+      mode="${mode}"
+      model="${model}"
+    />
   </xacro:unless>
 </robot>

File: dsr_description2/xacro/m0609.urdf.xacro (robot description, xacro)
@@ -5,7 +5,17 @@
   <xacro:arg name="namespace" default=""/>
   <xacro:arg name="use_gazebo" default="false"/>
+  <xacro:arg name="host" default=""/>
+  <xacro:arg name="port" default=""/>
+  <xacro:arg name="rt_host" default=""/>
+  <xacro:arg name="mode" default=""/>
+  <xacro:arg name="model" default=""/>
   <xacro:property name="gz" value="$(arg use_gazebo)"/>
   <xacro:property name="cr" value="$(arg color)"/>
   <xacro:property name="gr" value="$(arg gripper)"/>
+  <xacro:property name="host" value="$(arg host)"/>
+  <xacro:property name="rt_host" value="$(arg rt_host)"/>
+  <xacro:property name="port" value="$(arg port)"/>
+  <xacro:property name="mode" value="$(arg mode)"/>
+  <xacro:property name="model" value="$(arg model)"/>
   <xacro:if value="${cr == 'white'}">
      <xacro:include filename="$(find dsr_description2)/xacro/macro.m0609.white.xacro" />
@@ -28,5 +38,12 @@
   <xacro:unless value="${gz}">
     <xacro:include filename="$(find dsr_description2)/ros2_control/m0609.ros2_control.xacro" />
-    <xacro:m0609_ros2_control name="m0609"/>
+    <xacro:m0609_ros2_control
+      name="m0609"
+      host="${host}"
+      rt_host="${rt_host}"
+      port="${port}"
+      mode="${mode}"
+      model="${model}"
+    />
   </xacro:unless>
 </robot>

File: dsr_description2/xacro/m0617.urdf.xacro (robot description, xacro)
@@ -5,7 +5,17 @@
   <xacro:arg name="namespace" default=""/>
   <xacro:arg name="use_gazebo" default="false"/>
+  <xacro:arg name="host" default=""/>
+  <xacro:arg name="port" default=""/>
+  <xacro:arg name="rt_host" default=""/>
+  <xacro:arg name="mode" default=""/>
+  <xacro:arg name="model" default=""/>
   <xacro:property name="cr" value="$(arg color)"/>
   <xacro:property name="gr" value="$(arg gripper)"/>
   <xacro:property name="gz" value="$(arg use_gazebo)"/>
+  <xacro:property name="host" value="$(arg host)"/>
+  <xacro:property name="rt_host" value="$(arg rt_host)"/>
+  <xacro:property name="port" value="$(arg port)"/>
+  <xacro:property name="mode" value="$(arg mode)"/>
+  <xacro:property name="model" value="$(arg model)"/>
   <xacro:if value="${cr == 'white'}">
      <xacro:include filename="$(find dsr_description2)/xacro/macro.m0617.white.xacro" />
@@ -28,5 +38,12 @@
   <xacro:unless value="${gz}">
     <xacro:include filename="$(find dsr_description2)/ros2_control/m0617.ros2_control.xacro" />
-    <xacro:m0617_ros2_control name="m0617"/>
+    <xacro:m0617_ros2_control
+      name="m0617"
+      host="${host}"
+      rt_host="${rt_host}"
+      port="${port}"
+      mode="${mode}"
+      model="${model}"
+    />
   </xacro:unless>
 </robot>

File: dsr_description2/xacro/m1013.urdf.xacro (robot description, xacro)
@@ -5,7 +5,17 @@
   <xacro:arg name="namespace" default=""/>
   <xacro:arg name="use_gazebo" default="false"/>
+  <xacro:arg name="host" default=""/>
+  <xacro:arg name="port" default=""/>
+  <xacro:arg name="rt_host" default=""/>
+  <xacro:arg name="mode" default=""/>
+  <xacro:arg name="model" default=""/>
   <xacro:property name="cr" value="$(arg color)"/>
   <xacro:property name="gr" value="$(arg gripper)"/>
   <xacro:property name="gz" value="$(arg use_gazebo)"/>
+  <xacro:property name="host" value="$(arg host)"/>
+  <xacro:property name="rt_host" value="$(arg rt_host)"/>
+  <xacro:property name="port" value="$(arg port)"/>
+  <xacro:property name="mode" value="$(arg mode)"/>
+  <xacro:property name="model" value="$(arg model)"/>
   <xacro:if value="${cr == 'white'}">
      <xacro:include filename="$(find dsr_description2)/xacro/macro.m1013.white.xacro" />
@@ -28,5 +38,12 @@
   <xacro:unless value="${gz}">
     <xacro:include filename="$(find dsr_description2)/ros2_control/m1013.ros2_control.xacro" />
-    <xacro:m1013_ros2_control name="m1013"/>
+    <xacro:m1013_ros2_control
+      name="m1013"
+      host="${host}"
+      rt_host="${rt_host}"
+      port="${port}"
+      mode="${mode}"
+      model="${model}"
+    />
   </xacro:unless>
 </robot>

File: dsr_description2/xacro/m1509.urdf.xacro (robot description, xacro)
@@ -5,7 +5,17 @@
   <xacro:arg name="namespace" default=""/>
   <xacro:arg name="use_gazebo" default="false"/>
+  <xacro:arg name="host" default=""/>
+  <xacro:arg name="port" default=""/>
+  <xacro:arg name="rt_host" default=""/>
+  <xacro:arg name="mode" default=""/>
+  <xacro:arg name="model" default=""/>
   <xacro:property name="cr" value="$(arg color)"/>
   <xacro:property name="gr" value="$(arg gripper)"/>
   <xacro:property name="gz" value="$(arg use_gazebo)"/>
+  <xacro:property name="host" value="$(arg host)"/>
+  <xacro:property name="rt_host" value="$(arg rt_host)"/>
+  <xacro:property name="port" value="$(arg port)"/>
+  <xacro:property name="mode" value="$(arg mode)"/>
+  <xacro:property name="model" value="$(arg model)"/>
   <xacro:if value="${cr == 'white'}">
      <xacro:include filename="$(find dsr_description2)/xacro/macro.m1509.white.xacro" />
@@ -28,5 +38,12 @@
   <xacro:unless value="${gz}">
     <xacro:include filename="$(find dsr_description2)/ros2_control/m1509.ros2_control.xacro" />
-    <xacro:m1509_ros2_control name="m1509"/>
+    <xacro:m1509_ros2_control
+      name="m1509"
+      host="${host}"
+      rt_host="${rt_host}"
+      port="${port}"
+      mode="${mode}"
+      model="${model}"
+    />
   </xacro:unless>
 </robot>
