Commit message: Refactor controller  (#215)
* Refactor hw_interface & dsr_controller

* Fix launches as being changed workaround param to the standard way

File: dsr_description2/xacro/p3020.urdf.xacro (robot description, xacro)
@@ -5,7 +5,17 @@
   <xacro:arg name="namespace" default=""/>
   <xacro:arg name="use_gazebo" default="false"/>
+  <xacro:arg name="host" default=""/>
+  <xacro:arg name="port" default=""/>
+  <xacro:arg name="rt_host" default=""/>
+  <xacro:arg name="mode" default=""/>
+  <xacro:arg name="model" default=""/>
   <xacro:property name="cr" value="$(arg color)"/>
   <xacro:property name="gr" value="$(arg gripper)"/>
   <xacro:property name="gz" value="$(arg use_gazebo)"/>
+  <xacro:property name="host" value="$(arg host)"/>
+  <xacro:property name="rt_host" value="$(arg rt_host)"/>
+  <xacro:property name="port" value="$(arg port)"/>
+  <xacro:property name="mode" value="$(arg mode)"/>
+  <xacro:property name="model" value="$(arg model)"/>
   <xacro:if value="${cr == 'white'}">
      <xacro:include filename="$(find dsr_description2)/xacro/macro.p3020.white.xacro" />
@@ -28,5 +38,12 @@
   <xacro:unless value="${gz}">
     <xacro:include filename="$(find dsr_description2)/ros2_control/p3020.ros2_control.xacro" />
-    <xacro:p3020_ros2_control name="p3020"/>
+    <xacro:p3020_ros2_control
+      name="p3020"
+      host="${host}"
+      rt_host="${rt_host}"
+      port="${port}"
+      mode="${mode}"
+      model="${model}"
+    />
   </xacro:unless>
 </robot>
