Commit message: Add MuJoCo support feature. (#218)
* Add MuJoCo simulation feature

* Add red dot and scene for checking.

* Small tuning change for xml files

* Erase useless file, small change in XML files for test.

* Remove test code for gripper launch

* Add readme file

* Update readme

* Add license of 2f85, change readme

* Correct typo

* Add license mention on readme

* Now everything can be set in the main launch. Merge default and gripper launch file, new modul 'build_scene' added. Fix slope demo STL. + extra change

* Move objects dir to demo folder, change demo scene, correct license of dsr_mujoco, update readme

* Now support also H2017 blue, remove test example + extra tuning.

* Add brief doc

* Fix doc problem and update

* Update readme, erase useless files

* Update in readme

* Update doc

* Update readme (dependencies)

File: dsr_description2/xacro/h2017.urdf.xacro (robot description, xacro)
@@ -5,4 +5,5 @@
   <xacro:arg name="namespace" default=""/>
   <xacro:arg name="use_gazebo" default="false"/>
+  <xacro:arg name="use_mujoco" default="false"/>
   <xacro:arg name="host" default=""/>
   <xacro:arg name="port" default=""/>
@@ -13,4 +14,5 @@
   <xacro:property name="gr" value="$(arg gripper)"/>
   <xacro:property name="gz" value="$(arg use_gazebo)"/>
+  <xacro:property name="mj" value="$(arg use_mujoco)"/>
   <xacro:property name="host" value="$(arg host)"/>
   <xacro:property name="rt_host" value="$(arg rt_host)"/>
@@ -37,13 +39,20 @@
   </xacro:if>
   <xacro:unless value="${gz}">
-    <xacro:include filename="$(find dsr_description2)/ros2_control/h2017.ros2_control.xacro" />
-    <xacro:h2017_ros2_control
-      name="h2017"
-      host="${host}"
-      rt_host="${rt_host}"
-      port="${port}"
-      mode="${mode}"
-      model="${model}"
-    />
+    <!-- for mujoco -->
+    <xacro:if value="${mj}">
+      <xacro:include filename="$(find dsr_description2)/ros2_control/h2017.mj_ros2_control.xacro" />
+      <xacro:h2017_mj_ros2_control namespace="$(arg namespace)" gripper="$(arg gripper)"/>
+    </xacro:if>
+    <xacro:unless value="${mj}">
+      <xacro:include filename="$(find dsr_description2)/ros2_control/h2017.ros2_control.xacro" />
+      <xacro:h2017_ros2_control
+        name="h2017"
+        host="${host}"
+        rt_host="${rt_host}"
+        port="${port}"
+        mode="${mode}"
+        model="${model}"
+      />
+    </xacro:unless>
   </xacro:unless>
 </robot>

File: dsr_description2/xacro/m0609.urdf.xacro (robot description, xacro)
@@ -5,4 +5,5 @@
   <xacro:arg name="namespace" default=""/>
   <xacro:arg name="use_gazebo" default="false"/>
+  <xacro:arg name="use_mujoco" default="false"/>
   <xacro:arg name="host" default=""/>
   <xacro:arg name="port" default=""/>
@@ -10,7 +11,8 @@
   <xacro:arg name="mode" default=""/>
   <xacro:arg name="model" default=""/>
-  <xacro:property name="gz" value="$(arg use_gazebo)"/>
   <xacro:property name="cr" value="$(arg color)"/>
   <xacro:property name="gr" value="$(arg gripper)"/>
+  <xacro:property name="gz" value="$(arg use_gazebo)"/>
+  <xacro:property name="mj" value="$(arg use_mujoco)"/>
   <xacro:property name="host" value="$(arg host)"/>
   <xacro:property name="rt_host" value="$(arg rt_host)"/>
@@ -37,13 +39,20 @@
   </xacro:if>
   <xacro:unless value="${gz}">
-    <xacro:include filename="$(find dsr_description2)/ros2_control/m0609.ros2_control.xacro" />
-    <xacro:m0609_ros2_control
-      name="m0609"
-      host="${host}"
-      rt_host="${rt_host}"
-      port="${port}"
-      mode="${mode}"
-      model="${model}"
-    />
+    <!-- For mujoco -->
+    <xacro:if value="${mj}">
+      <xacro:include filename="$(find dsr_description2)/ros2_control/m0609.mj_ros2_control.xacro" />
+      <xacro:m0609_mj_ros2_control  namespace="$(arg namespace)" gripper="$(arg gripper)"/>
+    </xacro:if>
+    <xacro:unless value="${mj}">
+      <xacro:include filename="$(find dsr_description2)/ros2_control/m0609.ros2_control.xacro" />
+      <xacro:m0609_ros2_control
+        name="m0609"
+        host="${host}"
+        rt_host="${rt_host}"
+        port="${port}"
+        mode="${mode}"
+        model="${model}"
+      />
+    </xacro:unless>
   </xacro:unless>
 </robot>

File: dsr_description2/xacro/m1013.urdf.xacro (robot description, xacro)
@@ -5,4 +5,5 @@
   <xacro:arg name="namespace" default=""/>
   <xacro:arg name="use_gazebo" default="false"/>
+  <xacro:arg name="use_mujoco" default="false"/>
   <xacro:arg name="host" default=""/>
   <xacro:arg name="port" default=""/>
@@ -13,4 +14,5 @@
   <xacro:property name="gr" value="$(arg gripper)"/>
   <xacro:property name="gz" value="$(arg use_gazebo)"/>
+  <xacro:property name="mj" value="$(arg use_mujoco)"/>
   <xacro:property name="host" value="$(arg host)"/>
   <xacro:property name="rt_host" value="$(arg rt_host)"/>
@@ -37,13 +39,20 @@
   </xacro:if>
   <xacro:unless value="${gz}">
-    <xacro:include filename="$(find dsr_description2)/ros2_control/m1013.ros2_control.xacro" />
-    <xacro:m1013_ros2_control
-      name="m1013"
-      host="${host}"
-      rt_host="${rt_host}"
-      port="${port}"
-      mode="${mode}"
-      model="${model}"
-    />
+    <!-- for mujoco -->
+    <xacro:if value="${mj}">
+      <xacro:include filename="$(find dsr_description2)/ros2_control/m1013.mj_ros2_control.xacro" />
+      <xacro:m1013_mj_ros2_control namespace="$(arg namespace)" gripper="$(arg gripper)"/>
+    </xacro:if>
+    <xacro:unless value="${mj}">
+      <xacro:include filename="$(find dsr_description2)/ros2_control/m1013.ros2_control.xacro" />
+      <xacro:m1013_ros2_control
+        name="m1013"
+        host="${host}"
+        rt_host="${rt_host}"
+        port="${port}"
+        mode="${mode}"
+        model="${model}"
+      />
+    </xacro:unless>
   </xacro:unless>
 </robot>
