Commit message: Revise joint pose for M0609, M1509, M0617 and A0509 XACRO files. (#224)
* Update m1509 XACRO

* Update m0609 XACRO

* Upadte a0509 & m0617 XACRO files

File: dsr_description2/xacro/macro.a0509.blue.xacro (robot description, xacro)
@@ -31,5 +31,5 @@
 			<parent link="base_link" />
 			<child link="link_1" />
-			<origin rpy="0 0 0" xyz="0 0 0.1555" />
+			<origin rpy="0 0 0" xyz="0 0 0.1560" />
 			<axis xyz="0 0 1" />
 			<limit effort="194" lower="-6.2832" upper="6.2832" velocity="3.1416"/>

File: dsr_description2/xacro/macro.a0509.white.xacro (robot description, xacro)
@@ -31,5 +31,5 @@
 			<parent link="base_link" />
 			<child link="link_1" />
-			<origin rpy="0 0 0" xyz="0 0 0.1555" />
+			<origin rpy="0 0 0" xyz="0 0 0.1560" />
 			<axis xyz="0 0 1" />
 			<limit effort="194" lower="-6.2832" upper="6.2832" velocity="3.1416"/>

File: dsr_description2/xacro/macro.m0609.blue.xacro (robot description, xacro)
@@ -31,5 +31,5 @@
 			<parent link="base_link" />
 			<child link="link_1" />
-			<origin rpy="0 0 0" xyz="0 0 0.1" />
+			<origin rpy="0 0 0" xyz="0 0 0.1345" />
 			<axis xyz="0 0 1" />
 			<limit effort="163" lower="-6.2832" upper="6.2832" velocity="2.618"/>

File: dsr_description2/xacro/macro.m0609.white.xacro (robot description, xacro)
@@ -31,5 +31,5 @@
 			<parent link="base_link" />
 			<child link="link_1" />
-			<origin rpy="0 0 0" xyz="0 0 0.1" />
+			<origin rpy="0 0 0" xyz="0 0 0.1345" />
 			<axis xyz="0 0 1" />
 			<limit effort="163" lower="-6.2832" upper="6.2832" velocity="2.618"/>

File: dsr_description2/xacro/macro.m0617.blue.xacro (robot description, xacro)
@@ -31,5 +31,5 @@
 			<parent link="base_link" />
 			<child link="link_1" />
-			<origin rpy="0 0 0" xyz="0 0 0.1525" />
+			<origin rpy="0 0 0" xyz="0 0 0.1530" />
 			<axis xyz="0 0 1" />
 			<limit effort="346" lower="-6.2832" upper="6.2832" velocity="1.7453"/>

File: dsr_description2/xacro/macro.m0617.white.xacro (robot description, xacro)
@@ -31,5 +31,5 @@
 			<parent link="base_link" />
 			<child link="link_1" />
-			<origin rpy="0 0 0" xyz="0 0 0.1525" />
+			<origin rpy="0 0 0" xyz="0 0 0.1530" />
 			<axis xyz="0 0 1" />
 			<limit effort="346" lower="-6.2832" upper="6.2832" velocity="1.7453"/>

File: dsr_description2/xacro/macro.m1509.blue.xacro (robot description, xacro)
@@ -31,5 +31,5 @@
 			<parent link="base_link" />
 			<child link="link_1" />
-			<origin rpy="0 0 0" xyz="0 0 0.1525" />
+			<origin rpy="0 0 0" xyz="0 0 0.1530" />
 			<axis xyz="0 0 1" />
 			<limit effort="346" lower="-6.2832" upper="6.2832" velocity="2.618"/>

File: dsr_description2/xacro/macro.m1509.white.xacro (robot description, xacro)
@@ -31,5 +31,5 @@
 			<parent link="base_link" />
 			<child link="link_1" />
-			<origin rpy="0 0 0" xyz="0 0 0.1525" />
+			<origin rpy="0 0 0" xyz="0 0 0.1530" />
 			<axis xyz="0 0 1" />
 			<limit effort="346" lower="-6.2832" upper="6.2832" velocity="2.618"/>
