Commit message: Support m1509, m0617, h2515, a0509, a0912 and e0509 models in MuJoCo with ROS2. (#225)
* Add STL files for MuJoCo

* Add all model XACRO files and XML + some models scene files

* Add scene for all models and update XML files.

* Connect models to ROS2

* Tuned M1509

* Added density=”0” for clarification, tuned M0617

* Tuned H2525, A0509, A0912

* Tuned E0509

* Refactore new files, Remove test code, Remove P3020, Update README

* Update README

File: dsr_description2/xacro/a0509.urdf.xacro (robot description, xacro)
@@ -5,4 +5,5 @@
   <xacro:arg name="namespace" default=""/>
   <xacro:arg name="use_gazebo" default="false"/>
+  <xacro:arg name="use_mujoco" default="false"/>
   <xacro:arg name="host" default=""/>
   <xacro:arg name="port" default=""/>
@@ -13,4 +14,5 @@
   <xacro:property name="gr" value="$(arg gripper)"/>
   <xacro:property name="gz" value="$(arg use_gazebo)"/>
+  <xacro:property name="mj" value="$(arg use_mujoco)"/>
   <xacro:property name="host" value="$(arg host)"/>
   <xacro:property name="rt_host" value="$(arg rt_host)"/>
@@ -37,12 +39,20 @@
   </xacro:if>
   <xacro:unless value="${gz}">
-    <xacro:include filename="$(find dsr_description2)/ros2_control/a0509.ros2_control.xacro" />
-    <xacro:a0509_ros2_control name="a0509"
-      host="${host}"
-      rt_host="${rt_host}"
-      port="${port}"
-      mode="${mode}"
-      model="${model}"
-    />
+    <!-- for mujoco -->
+    <xacro:if value="${mj}">
+      <xacro:include filename="$(find dsr_description2)/ros2_control/a0509.mj_ros2_control.xacro" />
+      <xacro:a0509_mj_ros2_control namespace="$(arg namespace)" gripper="$(arg gripper)"/>
+    </xacro:if>
+    <xacro:unless value="${mj}">
+      <xacro:include filename="$(find dsr_description2)/ros2_control/a0509.ros2_control.xacro" />
+      <xacro:a0509_ros2_control
+        name="a0509"
+        host="${host}"
+        rt_host="${rt_host}"
+        port="${port}"
+        mode="${mode}"
+        model="${model}"
+      />
+    </xacro:unless>
   </xacro:unless>
 </robot>

File: dsr_description2/xacro/a0912.urdf.xacro (robot description, xacro)
@@ -5,4 +5,5 @@
   <xacro:arg name="namespace" default=""/>
   <xacro:arg name="use_gazebo" default="false"/>
+  <xacro:arg name="use_mujoco" default="false"/>
   <xacro:arg name="host" default=""/>
   <xacro:arg name="port" default=""/>
@@ -13,4 +14,5 @@
   <xacro:property name="gr" value="$(arg gripper)"/>
   <xacro:property name="gz" value="$(arg use_gazebo)"/>
+  <xacro:property name="mj" value="$(arg use_mujoco)"/>
   <xacro:property name="host" value="$(arg host)"/>
   <xacro:property name="rt_host" value="$(arg rt_host)"/>
@@ -37,12 +39,20 @@
   </xacro:if>
   <xacro:unless value="${gz}">
-    <xacro:include filename="$(find dsr_description2)/ros2_control/a0912.ros2_control.xacro" />
-    <xacro:a0912_ros2_control name="a0912"
-      host="${host}"
-      rt_host="${rt_host}"
-      port="${port}"
-      mode="${mode}"
-      model="${model}"
-    />
+    <!-- for mujoco -->
+    <xacro:if value="${mj}">
+      <xacro:include filename="$(find dsr_description2)/ros2_control/a0912.mj_ros2_control.xacro" />
+      <xacro:a0912_mj_ros2_control namespace="$(arg namespace)" gripper="$(arg gripper)"/>
+    </xacro:if>
+    <xacro:unless value="${mj}">
+      <xacro:include filename="$(find dsr_description2)/ros2_control/a0912.ros2_control.xacro" />
+      <xacro:a0912_ros2_control
+        name="a0912"
+        host="${host}"
+        rt_host="${rt_host}"
+        port="${port}"
+        mode="${mode}"
+        model="${model}"
+      />
+    </xacro:unless>
   </xacro:unless>
 </robot>

File: dsr_description2/xacro/e0509.urdf.xacro (robot description, xacro)
@@ -5,4 +5,5 @@
   <xacro:arg name="namespace" default=""/>
   <xacro:arg name="use_gazebo" default="false"/>
+  <xacro:arg name="use_mujoco" default="false"/>
   <xacro:arg name="host" default=""/>
   <xacro:arg name="port" default=""/>
@@ -13,4 +14,5 @@
   <xacro:property name="gr" value="$(arg gripper)"/>
   <xacro:property name="gz" value="$(arg use_gazebo)"/>
+  <xacro:property name="mj" value="$(arg use_mujoco)"/>
   <xacro:property name="host" value="$(arg host)"/>
   <xacro:property name="rt_host" value="$(arg rt_host)"/>
@@ -34,13 +36,20 @@
   </xacro:if>
   <xacro:unless value="${gz}">
-    <xacro:include filename="$(find dsr_description2)/ros2_control/e0509.ros2_control.xacro" />
-    <xacro:e0509_ros2_control
-      name="e0509"
-      host="${host}"
-      rt_host="${rt_host}"
-      port="${port}"
-      mode="${mode}"
-      model="${model}"
-    />
+    <!-- for mujoco -->
+    <xacro:if value="${mj}">
+      <xacro:include filename="$(find dsr_description2)/ros2_control/e0509.mj_ros2_control.xacro" />
+      <xacro:e0509_mj_ros2_control namespace="$(arg namespace)" gripper="$(arg gripper)"/>
+    </xacro:if>
+    <xacro:unless value="${mj}">
+      <xacro:include filename="$(find dsr_description2)/ros2_control/e0509.ros2_control.xacro" />
+      <xacro:e0509_ros2_control
+        name="e0509"
+        host="${host}"
+        rt_host="${rt_host}"
+        port="${port}"
+        mode="${mode}"
+        model="${model}"
+      />
+    </xacro:unless>
   </xacro:unless>
 </robot>

File: dsr_description2/xacro/h2515.urdf.xacro (robot description, xacro)
@@ -5,4 +5,5 @@
   <xacro:arg name="namespace" default=""/>
   <xacro:arg name="use_gazebo" default="false"/>
+  <xacro:arg name="use_mujoco" default="false"/>
   <xacro:arg name="host" default=""/>
   <xacro:arg name="port" default=""/>
@@ -13,4 +14,5 @@
   <xacro:property name="gr" value="$(arg gripper)"/>
   <xacro:property name="gz" value="$(arg use_gazebo)"/>
+  <xacro:property name="mj" value="$(arg use_mujoco)"/>
   <xacro:property name="host" value="$(arg host)"/>
   <xacro:property name="rt_host" value="$(arg rt_host)"/>
@@ -37,13 +39,20 @@
   </xacro:if>
   <xacro:unless value="${gz}">
-    <xacro:include filename="$(find dsr_description2)/ros2_control/h2515.ros2_control.xacro" />
-    <xacro:h2515_ros2_control
-      name="h2515"
-      host="${host}"
-      rt_host="${rt_host}"
-      port="${port}"
-      mode="${mode}"
-      model="${model}"
-    />
+    <!-- for mujoco -->
+    <xacro:if value="${mj}">
+      <xacro:include filename="$(find dsr_description2)/ros2_control/h2515.mj_ros2_control.xacro" />
+      <xacro:h2515_mj_ros2_control namespace="$(arg namespace)" gripper="$(arg gripper)"/>
+    </xacro:if>
+    <xacro:unless value="${mj}">
+      <xacro:include filename="$(find dsr_description2)/ros2_control/h2515.ros2_control.xacro" />
+      <xacro:h2515_ros2_control
+        name="h2515"
+        host="${host}"
+        rt_host="${rt_host}"
+        port="${port}"
+        mode="${mode}"
+        model="${model}"
+      />
+    </xacro:unless>
   </xacro:unless>
 </robot>

File: dsr_description2/xacro/m0617.urdf.xacro (robot description, xacro)
@@ -5,4 +5,5 @@
   <xacro:arg name="namespace" default=""/>
   <xacro:arg name="use_gazebo" default="false"/>
+  <xacro:arg name="use_mujoco" default="false"/>
   <xacro:arg name="host" default=""/>
   <xacro:arg name="port" default=""/>
@@ -13,4 +14,5 @@
   <xacro:property name="gr" value="$(arg gripper)"/>
   <xacro:property name="gz" value="$(arg use_gazebo)"/>
+  <xacro:property name="mj" value="$(arg use_mujoco)"/>
   <xacro:property name="host" value="$(arg host)"/>
   <xacro:property name="rt_host" value="$(arg rt_host)"/>
@@ -37,13 +39,20 @@
   </xacro:if>
   <xacro:unless value="${gz}">
-    <xacro:include filename="$(find dsr_description2)/ros2_control/m0617.ros2_control.xacro" />
-    <xacro:m0617_ros2_control
-      name="m0617"
-      host="${host}"
-      rt_host="${rt_host}"
-      port="${port}"
-      mode="${mode}"
-      model="${model}"
-    />
+    <!-- for mujoco -->
+    <xacro:if value="${mj}">
+      <xacro:include filename="$(find dsr_description2)/ros2_control/m0617.mj_ros2_control.xacro" />
+      <xacro:m0617_mj_ros2_control namespace="$(arg namespace)" gripper="$(arg gripper)"/>
+    </xacro:if>
+    <xacro:unless value="${mj}">
+      <xacro:include filename="$(find dsr_description2)/ros2_control/m0617.ros2_control.xacro" />
+      <xacro:m0617_ros2_control
+        name="m0617"
+        host="${host}"
+        rt_host="${rt_host}"
+        port="${port}"
+        mode="${mode}"
+        model="${model}"
+      />
+    </xacro:unless>
   </xacro:unless>
 </robot>

File: dsr_description2/xacro/m1509.urdf.xacro (robot description, xacro)
@@ -5,4 +5,5 @@
   <xacro:arg name="namespace" default=""/>
   <xacro:arg name="use_gazebo" default="false"/>
+  <xacro:arg name="use_mujoco" default="false"/>
   <xacro:arg name="host" default=""/>
   <xacro:arg name="port" default=""/>
@@ -13,4 +14,5 @@
   <xacro:property name="gr" value="$(arg gripper)"/>
   <xacro:property name="gz" value="$(arg use_gazebo)"/>
+  <xacro:property name="mj" value="$(arg use_mujoco)"/>
   <xacro:property name="host" value="$(arg host)"/>
   <xacro:property name="rt_host" value="$(arg rt_host)"/>
@@ -37,13 +39,20 @@
   </xacro:if>
   <xacro:unless value="${gz}">
-    <xacro:include filename="$(find dsr_description2)/ros2_control/m1509.ros2_control.xacro" />
-    <xacro:m1509_ros2_control
-      name="m1509"
-      host="${host}"
-      rt_host="${rt_host}"
-      port="${port}"
-      mode="${mode}"
-      model="${model}"
-    />
+    <!-- for mujoco -->
+    <xacro:if value="${mj}">
+      <xacro:include filename="$(find dsr_description2)/ros2_control/m1509.mj_ros2_control.xacro" />
+      <xacro:m1509_mj_ros2_control namespace="$(arg namespace)" gripper="$(arg gripper)"/>
+    </xacro:if>
+    <xacro:unless value="${mj}">
+      <xacro:include filename="$(find dsr_description2)/ros2_control/m1509.ros2_control.xacro" />
+      <xacro:m1509_ros2_control
+        name="m1509"
+        host="${host}"
+        rt_host="${rt_host}"
+        port="${port}"
+        mode="${mode}"
+        model="${model}"
+      />
+    </xacro:unless>
   </xacro:unless>
 </robot>

File: dsr_description2/xacro/p3020.urdf.xacro (robot description, xacro)
@@ -5,4 +5,5 @@
   <xacro:arg name="namespace" default=""/>
   <xacro:arg name="use_gazebo" default="false"/>
+  <xacro:arg name="use_mujoco" default="false"/>
   <xacro:arg name="host" default=""/>
   <xacro:arg name="port" default=""/>
@@ -13,4 +14,5 @@
   <xacro:property name="gr" value="$(arg gripper)"/>
   <xacro:property name="gz" value="$(arg use_gazebo)"/>
+  <xacro:property name="mj" value="$(arg use_mujoco)"/>
   <xacro:property name="host" value="$(arg host)"/>
   <xacro:property name="rt_host" value="$(arg rt_host)"/>
@@ -33,17 +35,24 @@
   </joint>
   <xacro:if value="${gz}">
-    <xacro:include filename="$(find dsr_description2)/ros2_control/p3020.gz_ros2_control.xacro" />
-    <xacro:p3020_gz_ros2_control namespace="$(arg namespace)"/>
+    <xacro:include filename="$(find dsr_description2)/ros2_control/m1509.gz_ros2_control.xacro" />
+    <xacro:m1509_gz_ros2_control namespace="$(arg namespace)"/>
   </xacro:if>
   <xacro:unless value="${gz}">
-    <xacro:include filename="$(find dsr_description2)/ros2_control/p3020.ros2_control.xacro" />
-    <xacro:p3020_ros2_control
-      name="p3020"
-      host="${host}"
-      rt_host="${rt_host}"
-      port="${port}"
-      mode="${mode}"
-      model="${model}"
-    />
+    <!-- for mujoco -->
+    <xacro:if value="${mj}">
+      <xacro:include filename="$(find dsr_description2)/ros2_control/m1509.mj_ros2_control.xacro" />
+      <xacro:m1509_mj_ros2_control namespace="$(arg namespace)" gripper="$(arg gripper)"/>
+    </xacro:if>
+    <xacro:unless value="${mj}">
+      <xacro:include filename="$(find dsr_description2)/ros2_control/m1509.ros2_control.xacro" />
+      <xacro:m1509_ros2_control
+        name="m1509"
+        host="${host}"
+        rt_host="${rt_host}"
+        port="${port}"
+        mode="${mode}"
+        model="${model}"
+      />
+    </xacro:unless>
   </xacro:unless>
 </robot>
